File: Kicad/Esp32WROOM/Esp32Wroom.kicad_sch (KiCad schematic)
At the start: 31 parts, among them J1 Conn_01x03_Pin, J2 Conn_01x03_Socket, J3 Conn_01x08_Pin, J4 Conn_01x08_Socket, J5 Conn_01x02_Pin, M1 Motor_DC, Q1 TIP120, Q2 TIP120, Q3 TIP120, Q4 TIP120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

Commit message: aggiornato kicad
Parts:
- removed J5: Conn_01x02_Pin, symbol Connector:Conn_01x02_Pin
- removed M1: Motor_DC, symbol Motor:Motor_DC
- removed Q6, Q7: TIP120, Package_TO_SOT_THT:TO-220-3_Vertical, symbol Transistor_BJT:TIP120
- removed R8, R9: 1k, Resistor_THT:R_Axial_DIN0204_L3.6mm_D1.6mm_P5.08mm_Horizontal, symbol Device:R
- removed U3: 4N25, Package_DIP:DIP-6_W7.62mm, symbol Isolator:4N25
Connections:
- no-connect marks 5 -> 4
Other:
- note added: "ESP32-S3 mini per con: Sensore temperatura Sensore umidità Sensore luminosità Pilotaggio n. 4 led 3W con darlington in unico case Pilotaggio led Ultravioletto 1W N. 3 pulsanti touch N. 1 displat ST7789 SPI"
- note removed: "ESP32-C3 per terrario iMac con: Sensore temperatura Sensore umidità Sensore luminosità Pilotaggio n. 6 led 3W con darlington Controllo pomap acqua Controllo effetto nebbia"

Commit message: uff01
Parts:
- removed D4, D5, D6: LED, symbol Device:LED
- removed J3: Conn_01x08_Pin, symbol Connector:Conn_01x08_Pin
- removed J4: Conn_01x08_Socket, symbol Connector:Conn_01x08_Socket
- removed Q4, Q5: TIP120, Package_TO_SOT_THT:TO-220-3_Vertical, symbol Transistor_BJT:TIP120
- removed R6, R7: 1k, Resistor_THT:R_Axial_DIN0204_L3.6mm_D1.6mm_P5.08mm_Horizontal, symbol Device:R
- removed U1: ESP32-C3, ESP32-C3-WROOM, symbol RF_Module:ESP32-C3-WROOM-02U
- added J3: Conn_01x04_Pin, symbol Connector:Conn_01x04_Pin
- added J5: Conn_01x04_Socket, symbol Connector:Conn_01x04_Socket
- added U3: ESP32-S3-Mini, ESP32-C3-WROOM, symbol New_Library:ESP32-S3-Mini
Connections:
- net +3.3V: now also U3.3 (3V3)
- net +5V: now also J5.1 (Pin_1), U3.1 (5V)
- net DHT: now also U3.8 (IO09)
- net FOG1: now also U3.14 (I003)
- net GND: now also U3.2 (GND)
- net LED1: now also U3.7 (IO10)
- net LED2: now also U3.5 (IO12)
- net LED3: now also U3.4 (IO13)
- net LED6: now also U3.16 (IO01)
- net M1: now also U3.15 (I002)
- net at Q1.2 (C): now also J5.2 (Pin_2)
- net at D1.1 (K), D2.1 (K), D3.1 (K): now also J3.1 (Pin_1)
- net at D3.2 (A): now also J3.4 (Pin_4)
- net at Q2.2 (C): now also J5.3 (Pin_3)
- net at R1.2, R2.1: now also U3.6 (IO11)
- net at D2.2 (A): now also J3.3 (Pin_3)
- net at D1.2 (A): now also J3.2 (Pin_2)
- net at Q3.2 (C): now also J5.4 (Pin_4)
- no-connect marks 4 -> 1
Other:
- note added: "ESP32-S3 mini per con: Sensore temperatura Sensore umidità Sensore luminosità Pilotaggio n. 3 led 3W con darlington N. 3 pulsanti N. 1 display ST7789 SPI"
- note removed: "ESP32-S3 mini per con: Sensore temperatura Sensore umidità Sensore luminosità Pilotaggio n. 4 led 3W con darlington in unico case Pilotaggio led Ultravioletto 1W N. 3 pulsanti touch N. 1 displat ST7789 SPI"
- title: (none) -> Terrario conS3 Mini

Commit message: uff01
Parts:
- removed J1: Conn_01x03_Pin, symbol Connector:Conn_01x03_Pin
- removed J2: Conn_01x03_Socket, symbol Connector:Conn_01x03_Socket
- removed J3: Conn_01x04_Pin, symbol Connector:Conn_01x04_Pin
- removed J5: Conn_01x04_Socket, symbol Connector:Conn_01x04_Socket
- removed U3: ESP32-S3-Mini, ESP32-C3-WROOM, symbol New_Library:ESP32-S3-Mini
- added D4: G, symbol Device:LED
- added D5: UV, symbol Device:LED
- added J1: Conn_01x08_Socket, symbol Connector:Conn_01x08_Socket
- added J2: Conn_01x08_Pin, symbol Connector:Conn_01x08_Pin
- added J3: Conn_01x10_Socket, symbol Connector:Conn_01x10_Socket
- added J4: Conn_01x10_Pin, symbol Connector:Conn_01x10_Pin
- added J5: Conn_01x05_Socket, symbol Connector:Conn_01x05_Socket
- added J6: Conn_01x02_Socket, symbol Connector:Conn_01x02_Socket
- added J7: Conn_01x05_Pin, symbol Connector:Conn_01x05_Pin
- added J8: Conn_01x02_Pin, symbol Connector:Conn_01x02_Pin
- added M1: Fan, symbol Motor:Fan
- added Q4, Q5, Q6: TIP120, Package_TO_SOT_THT:TO-220-3_Vertical, symbol Transistor_BJT:TIP120
- added R5, R6, R7: 1k, Resistor_THT:R_Axial_DIN0204_L3.6mm_D1.6mm_P5.08mm_Horizontal, symbol Device:R
- added SW1: <, symbol Switch:SW_Push
- added SW2: Ok, symbol Switch:SW_Push
- added SW3: >, symbol Switch:SW_Push
- added U1: ESP32-WROOM, ESP32 30 pin, symbol Esp32-rescue:ESP32-WROOM
- added U2: ST7789, ST7789, symbol Esp32-rescue:ST7789
- D1: value LED -> W
- D2: value LED -> R
- D3: value LED -> B
- renumbered R3 to R2, R4 to R3, R5 to R4, R2 to R8, U2 to U3
Connections:
- net +3.3V: now also R1.2, J1.2 (Pin_2), J3.8 (Pin_8), U1.1 (3.3V); no longer R1.1
- net +5V: now also J3.1 (Pin_1), J6.1 (Pin_1), J8.1 (Pin_1), U1.30 (VIN)
- net DHT: now also J3.9 (Pin_9), U1.7 (IO17)
- net GND: now also J1.1 (Pin_1), J3.10 (Pin_10), J5.5 (Pin_5), J6.2 (Pin_2), J8.2 (Pin_2), Q4.3 (E), Q5.3 (E), Q6.3 (E), U1.32 (GND); no longer R8.2
- net at D1.1 (K), D2.1 (K), D3.1 (K): now also D4.1 (K), D5.1 (K), J4.1 (Pin_1), M1.1 (+)
- net at D1.2 (A): now also J4.2 (Pin_2)
- net at D2.2 (A): now also J4.3 (Pin_3)
- net at D3.2 (A): now also J4.4 (Pin_4)
- net at U3.1 (VDD): now also J4.8 (Pin_8)
- net at U3.2 (DATA): now also J4.9 (Pin_9)
- net at U3.4 (GND): now also J4.10 (Pin_10)
- net at Q1.2 (C): now also J3.2 (Pin_2)
- net at Q2.2 (C): now also J3.3 (Pin_3)
- net at Q3.2 (C): now also J3.4 (Pin_4)
- net at R8.1: now also J7.4 (Pin_4); no longer R1.2
- net LED1 renamed LED_W
- net LED_W: now also U1.25 (IO27)
- net LED2 renamed LED_R
- net LED_R: now also U1.23 (IO25)
- net LED3 renamed LED_B
- net LED_B: now also U1.14 (IO22)
- new net: J2.1 (Pin_1), U2.1 (GND)
- new net: J2.2 (Pin_2), U2.2 (3.3V)
- new net: J2.3 (Pin_3), U2.3 (SCL)
- new net: J2.4 (Pin_4), U2.4 (SDA)
- new net: J2.5 (Pin_5), U2.5 (RES)
- new net: J2.6 (Pin_6), U2.6 (DC)
- new net: J2.7 (Pin_7), U2.7 (CS)
- new net: J2.8 (Pin_8), U2.8 (BLK)
- new net: D4.2 (A), J4.5 (Pin_5)
- new net: D5.2 (A), J4.6 (Pin_6)
- new net: J4.7 (Pin_7), M1.2 (-)
- new net: J7.1 (Pin_1), SW1.1
- new net: J7.2 (Pin_2), SW2.1
- new net: J7.3 (Pin_3), SW3.1
- new net: J7.5 (Pin_5), R8.2, SW1.2, SW2.2, SW3.2
- new net: Q4.1 (B), R5.2
- new net: J3.5 (Pin_5), Q4.2 (C)
- new net: J3.6 (Pin_6), Q5.2 (C)
- new net: J3.7 (Pin_7), Q6.2 (C)
- new net: Q6.1 (B), R7.2
- new net: Q5.1 (B), R6.2
- new net <: J5.1 (Pin_1), U1.28 (IO13)
- new net >: J5.3 (Pin_3), U1.26 (IO14)
- new net BLK: J1.8 (Pin_8), U1.11 (IO21)
- new net CS: J1.7 (Pin_7), U1.9 (IO18)
- new net DC: J1.6 (Pin_6), U1.15 (IO23)
- new net FAN: R7.1, U1.24 (IO26)
- new net LED_G: R5.1, U1.21 (IO32)
- new net LED_UV: R6.1, U1.22 (IO33)
- new net OK: J5.2 (Pin_2), U1.3 (IO15)
- new net PHOTO: J5.4 (Pin_4), R1.1, U1.20 (IO35)
- new net RES: J1.5 (Pin_5), U1.10 (IO19)
- new net SCL: J1.3 (Pin_3), U1.6 (IO16)
- new net SDA: J1.4 (Pin_4), U1.8 (IO05)
- no-connect marks 1 -> 10
Other:
- note added: "ESP32-WROOM 30 pin per con: Sensore temperatura Sensore umidità Sensore luminosità Pilotaggio n. 3 led 3W con darlington Pilotaggio 1 led UV Pilotaggio PWD ventola N. 3 pulsanti N. 1 display ST7789 SPI"
- note removed: "ESP32-S3 mini per con: Sensore temperatura Sensore umidità Sensore luminosità Pilotaggio n. 3 led 3W con darlington N. 3 pulsanti N. 1 display ST7789 SPI"
- title: Terrario conS3 Mini -> Terrario con ESP32 30 pin
- moved on the sheet: D1, D2, D3, Q1, Q2, Q3, R1, R2, R3, R4, R8, U3
